File: HW/esp32_charger/scheme.brd (EAGLE design)
At the start: 100 x 80 mm, 23 parts, among them IC3 24C01SN, K1 4052, T1 2N7002E, T2 2N7002E

Commit message: Updated project and gitignore
Parts:
- added C2: 10uF, rcl:C0805
- added C2-TANT: 22uF, rcl:C3216
- added IC1: LM1117IMPX-3.3, lm1117:SOT223
- added LED1: (no value), led:CHIP-LED0805
- added R9: 500, rcl:R0805
- added SV2: (no value), con-lstb:MA03-1
Connections:
- new net +3V3: C2-TANT.1, IC1.2, IC1.TAB, U$1.1
- new net +5V: C2.1, IC1.3, R9.2, SV2.2
- new net N$1: LED1.A, R9.1
- net GND: now also C2-TANT.2, C2.2, IC1.1, LED1.C, SV2.1
- net VCC: no longer U$1.1
Changed lines of the file:
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@@
 <?xml version="1.0" encoding="utf-8"?>
 <!DOCTYPE eagle SYSTEM "eagle.dtd">
-<eagle version="9.3.2">
+<eagle version="9.4.2">
 <drawing>
 <settings>
@@
 <layer number="230" name="230bmp" color="7" fill="1" visible="yes" active="yes"/>
 <layer number="231" name="231bmp" color="7" fill="1" visible="yes" active="yes"/>
+<layer number="232" name="Eagle3D_PG2" color="7" fill="1" visible="no" active="no"/>
+<layer number="233" name="Eagle3D_PG3" color="7" fill="1" visible="no" active="no"/>
 <layer number="248" name="Housing" color="7" fill="1" visible="yes" active="yes"/>
 <layer number="249" name="Edge" color="7" fill="1" visible="yes" active="yes"/>
@@
 <attribute name="VALUE" x="-56.769" y="-129.921" size="0.8128" layer="21" font="vector" ratio="15"/>
 </element>
+<element name="IC1" library="lm1117" package="SOT223" value="LM1117IMPX-3.3" x="-35.56" y="-144.78" smashed="yes">
+<attribute name="NAME" x="-39.4208" y="-146.05" size="1.27" layer="25" rot="R90"/>
+<attribute name="VALUE" x="-30.4292" y="-146.05" size="1.27" layer="27" rot="R90"/>
+</element>
+<element name="SV2" library="con-lstb" library_urn="urn:adsk.eagle:library:162" package="MA03-1" package3d_urn="urn:adsk.eagle:package:8339/1" value="" x="-54.61" y="-171.45" smashed="yes">
+<attribute name="MF" value="" x="-73.66" y="-147.32" size="1.778" layer="27" display="off"/>
+<attribute name="MPN" value="" x="-73.66" y="-147.32" size="1.778" layer="27" display="off"/>
+<attribute name="NAME" x="-58.42" y="-169.799" size="1.27" layer="25" ratio="10"/>
+<attribute name="OC_FARNELL" value="unknown" x="-73.66" y="-147.32" size="1.778" layer="27" display="off"/>
+<attribute name="OC_NEWARK" value="unknown" x="-73.66" y="-147.32" size="1.778" layer="27" display="off"/>
+<attribute name="VALUE" x="-58.42" y="-174.371" size="1.27" layer="27" ratio="10"/>
+</element>
+<element name="C2" library="rcl" library_urn="urn:adsk.eagle:library:334" package="C0805" package3d_urn="urn:adsk.eagle:package:23617/2" value="10uF" x="-49.53" y="-163.83" smashed="yes">
+<attribute name="NAME" x="-50.8" y="-162.56" size="1.27" layer="25"/>
+<attribute name="SPICEPREFIX" value="C" x="-77.47" y="-152.4" size="1.778" layer="27" display="off"/>
+<attribute name="VALUE" x="-50.8" y="-166.37" size="1.27" layer="27"/>
+</element>
+<element name="C2-TANT" library="rcl" library_urn="urn:adsk.eagle:library:334" package="C3216" package3d_urn="urn:adsk.eagle:package:23628/2" value="22uF" x="-58.42" y="-163.83" smashed="yes">
+<attribute name="NAME" x="-59.69" y="-162.56" size="1.27" layer="25"/>
+<attribute name="SPICEPREFIX" value="C" x="-77.47" y="-158.75" size="1.778" layer="27" display="off"/>
+<attribute name="VALUE" x="-59.69" y="-166.37" size="1.27" layer="27"/>
+</element>
+<element name="R9" library="rcl" library_urn="urn:adsk.eagle:library:334" package="R0805" package3d_urn="urn:adsk.eagle:package:23553/2" value="500" x="-43.18" y="-163.83" smashed="yes">
+<attribute name="NAME" x="-43.815" y="-162.56" size="1.27" layer="25"/>
+<attribute name="SPICEPREFIX" value="R" x="-77.47" y="-165.1" size="1.778" layer="27" display="off"/>
+<attribute name="VALUE" x="-43.815" y="-166.37" size="1.27" layer="27"/>
+</element>
+<element name="LED1" library="led" library_urn="urn:adsk.eagle:library:259" package="CHIP-LED0805" package3d_urn="urn:adsk.eagle:package:15818/2" value="" x="-36.83" y="-163.83" smashed="yes">
+<attribute name="NAME" x="-38.1" y="-165.1" size="1.27" layer="25" rot="R90"/>
+<attribute name="VALUE" x="-34.29" y="-165.1" size="1.27" layer="27" rot="R90"/>
+</element>
 </elements>
 <signals>
@@
 <contactref element="IC3" pad="7"/>
 <contactref element="IC3" pad="4"/>
-<wire x1="-56.515" y1="-110.55" x2="-57.785" y2="-110.55" width="0" layer="19" extent="1-1"/>
-<wire x1="-55.245" y1="-110.55" x2="-56.515" y2="-110.55" width="0" layer="19" extent="1-1"/>
-<wire x1="-53.975" y1="-110.55" x2="-55.245" y2="-110.55" width="0" layer="19" extent="1-1"/>
+<contactref element="IC1" pad="1"/>
+<contactref element="SV2" pad="1"/>
+<contactref element="LED1" pad="C"/>
+<contactref element="C2" pad="2"/>
+<contactref element="C2-TANT" pad="2"/>
+<wire x1="-57.02" y1="-163.83" x2="-57.15" y2="-171.45" width="0" layer="19" extent="1-1"/>
+<wire x1="-48.58" y1="-163.83" x2="-57.02" y2="-163.83" width="0" layer="19" extent="1-1"/>
+<wire x1="-36.83" y1="-162.78" x2="-48.58" y2="-163.83" width="0" layer="19" extent="1-1"/>
+<wire x1="-37.871" y1="-147.879" x2="-36.83" y2="-162.78" width="0" layer="19" extent="1-1"/>
+<wire x1="-53.975" y1="-110.55" x2="-37.871" y2="-147.879" width="0" layer="19" extent="1-1"/>
+<wire x1="-55.245" y1="-110.55" x2="-53.975" y2="-110.55" width="0" layer="19" extent="1-1"/>
+<wire x1="-56.515" y1="-110.55" x2="-55.245" y2="-110.55" width="0" layer="19" extent="1-1"/>
+<wire x1="-57.785" y1="-110.55" x2="-56.515" y2="-110.55" width="0" layer="19" extent="1-1"/>
 <wire x1="-56.515" y1="-105.35" x2="-56.515" y2="-110.55" width="0" layer="19" extent="1-1"/>
 <wire x1="-46.99" y1="-86.36" x2="-56.515" y2="-105.35" width="0" layer="19" extent="1-1"/>
@@
 <signal name="VCC">
 <contactref element="U$3" pad="2"/>
-<contactref element="U$1" pad="1"/>
 <contactref element="R6" pad="P$1"/>
 <contactref element="IC3" pad="8"/>
@@
 <wire x1="-59.69" y1="-99.06" x2="-57.785" y2="-105.35" width="0" layer="19" extent="1-1"/>
 <wire x1="-43.18" y1="30.48" x2="-59.69" y2="-99.06" width="0" layer="19" extent="1-1"/>
-<wire x1="25.39" y1="23.29" x2="-43.18" y2="30.48" width="0" layer="19" extent="1-1"/>
 </signal>
 <signal name="N$3">
@@
 <wire x1="58.41" y1="23.29" x2="-26.035" y2="20.32" width="0" layer="19" extent="1-1"/>
 </signal>
+<signal name="+5V">
+<contactref element="IC1" pad="3"/>
+<contactref element="SV2" pad="2"/>
+<contactref element="R9" pad="2"/>
+<contactref element="C2" pad="1"/>
+<wire x1="-50.48" y1="-163.83" x2="-54.61" y2="-171.45" width="0" layer="19" extent="1-1"/>
+<wire x1="-42.23" y1="-163.83" x2="-50.48" y2="-163.83" width="0" layer="19" extent="1-1"/>
+<wire x1="-33.249" y1="-147.879" x2="-42.23" y2="-163.83" width="0" layer="19" extent="1-1"/>
+</signal>
+<signal name="+3V3">
+<contactref element="IC1" pad="2"/>
+<contactref element="IC1" pad="TAB"/>
+<contactref element="C2-TANT" pad="1"/>
+<contactref element="U$1" pad="1"/>
+<wire x1="-35.56" y1="-147.879" x2="-59.82" y2="-163.83" width="0" layer="19" extent="1-1"/>
+<wire x1="-35.56" y1="-141.681" x2="-35.56" y2="-147.879" width="0" layer="19" extent="1-1"/>
+<wire x1="25.39" y1="23.29" x2="-35.56" y2="-141.681" width="0" layer="19" extent="1-1"/>
+</signal>
+<signal name="N$1">
+<contactref element="R9" pad="1"/>
+<contactref element="LED1" pad="A"/>
+<wire x1="-36.83" y1="-164.88" x2="-44.13" y2="-163.83" width="0" layer="19" extent="1-1"/>
+</signal>
 </signals>

Commit message: Added bare esp32 and ds1307
Parts:
- removed 12V, PZEM004T_POWER, PZEM004T_RX_TX: (no value), antduino:SPARKFUN_1X02
- removed DS1307: RTC-EEPROM-BATTERY, diy-modules:RTC-EEPROM-BATTERY
- removed IC1: LM1117IMPX-3.3, lm1117:SOT223
- removed U$1: ESP32DEVKITV1, ESP32-DEVKITV1:ESP32-DEVKITV1
- added BT1: ML-1220/F1AN, batteries:ML-1220/F1BN
- added D3: SM4007, _mod_diode:MELF-MLL41
- added IC2: DS1307Z, ds1307_pcf8583:SOIC8
- added IC4: LM1117IDTX-3.3, lm1117:TO252
- added R10: 200, rcl:R0805
- added R11, R13, R14: 3.3K, rcl:R0805
- added R12: 510K, rcl:R0805
- added R15: 1.5M, rcl:R0805
- added U1: ESP3212, esp32:ESP3212
- added X1: CRYSTALS-NOGND-WATCH-3X8, IQD-Frequency-Products:WATCH-3X8
- R6: value 10K-100K -> 10K
- SV2: value (none) -> 12V
Connections:
- removed net +5V: C2.1, IC1.3, R9.2, SV2.2
- removed net GND.2: DS1307.J2.2
- removed net N$3: DS1307.J1.2, PZEM004T_POWER.1, U$1.30
- removed net N$4: PZEM004T_RX_TX.1, U$1.7
- removed net N$5: PZEM004T_RX_TX.2, U$1.6
- removed net N$7: 12V.2, C1.1, D2.C, K1.1, R1.P$2
- removed net VCC.2: DS1307.J2.3
- new net N$16: IC2.2, X1.1
- new net N$17: IC2.6, IC3.6, R14.1, R8.P$1, U$3.3, U1.27
- new net N$18: IC2.5, IC3.5, R13.1, R7.P$1, U$3.4, U1.30
- new net N$19: IC2.3, R12.2, R15.2
- new net N$2: IC2.1, X1.2
- new net N$20: BT1.POS, D3.C, R12.1
- net +3V3: now also IC2.8, IC3.8, IC4.TAB, R10.1, R11.1, R13.2, R14.2, R6.P$1, R7.P$2, R8.P$2, U$3.2, U1.21; no longer IC1.2, IC1.TAB, U$1.1
- net GND: now also BT1.NEG, IC2.4, IC4.1, R15.1, U1.1, U1.16, U1.31; no longer 12V.1, DS1307.J1.1, IC1.1, PZEM004T_POWER.2, U$1.2
- net N$11: now also U1.3; no longer U$1.17
- net N$14: now also U1.9; no longer U$1.23
- net N$15: now also IC2.7, R11.2; no longer DS1307.J1.4, IC3.6, R8.P$1, U$1.14, U$3.3
- net N$22: now also D3.A, R10.2; no longer DS1307.J1.3, IC3.5, R7.P$1, U$1.11, U$3.4
- net N$6: now also U1.8; no longer U$1.22
- net N$9: now also U1.7; no longer U$1.21
- net VCC: now also C1.1, C2.1, D2.C, IC4.2, K1.1, R1.P$2, R9.2, SV2.2; no longer IC3.8, R6.P$1, R7.P$2, R8.P$2, U$3.2
